File: MiniDrone_FC.kicad_pcb (KiCad board)
At the start: 2 copper layers, 76.6 x 76.6 mm, 60 parts, among them J1 BATT 1S, J2 USB-C, J3 DEBUG, M1 Motor CW, M2 Motor CCW, M3 Motor CCW, M4 Motor CW, Q1 AO3400A, Q2 AO3400A, Q3 AO3400A, Q4 AO3400A, Q5 AO3401A, SW1 RESET, SW2 BOOT, U1 ESP32-S3-WROOM-1-N8, U2 AP2112K-3.3, U3 MPU-6050

Commit message: silk screen update
Other:
- board text added: "GNX Works"
- board text removed: "GNX Robotics"
Changed lines of the file:
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@@
 		)
 	)
-	(gr_text "GNX Robotics"
+	(gr_text "GNX Works"
 		(at 139 121.5 0)
 		(layer "B.SilkS")
